File: kicad/sp7021-block/sp7021-block.kicad_sch (KiCad schematic)
At the start: 72 parts

Commit message: Sep 26, 2024 2
Parts:
- removed C? (x2): 22uF, symbol Device:C_Small
- removed C?: 10uF, symbol Device:C_Small
- removed C?: 100nF, symbol Device:C_Small
- removed L?: 3.9uH, symbol Device:L_Small
- removed U?: AP63203WU, Package_TO_SOT_SMD:TSOT-23-6, symbol sp7021-block:AP63203WU
- added U?: TPS65400, Package_DFN_QFN:Texas_RGZ0048A_VQFN-48-1EP_7x7mm_P0.5mm_EP5.15x5.15mm_ThermalVias, symbol sp7021-block:TPS65400
Connections:
- net SYS_5V: now reaches C?.1, C?.1, C?.1, C?.1, L?.2, R?.1, R?.1
- net SYS_5V: no longer U?.1 (IN), U?.1 (IN)
- new net: U?.10 (SW2), U?.11 (SW2), U?.9 (SW2)
- new net: U?.2 (SW1), U?.3 (SW1), U?.4 (SW1)
- new net: U?.1 (IN), U?.1 (IN)
Other:
- moved on the sheet: C?, L?, R?, U?, U?I, U?J

Commit message: Oct 14, 2024
Parts:
- removed R? (x2): 2.2K, symbol Device:R_Small
- added C? (x4): 100nF, symbol Device:C_Small
- added C? (x2): 15pF, Capacitor_SMD:C_0603_1608Metric, symbol Device:C_Small
- added C?: 10uF, symbol Device:C_Small
- added C?: 2.2uF, symbol Device:C_Small
- added D?: BAT201M3, Diode_SMD:D_SOD-323F, symbol Device:D_Schottky_Small_Filled
- added J?: Debug, symbol Connector_Generic:Conn_01x03
- added J?: Conn_01x02, symbol Connector_Generic:Conn_01x02
- added J?: Conn_01x40, symbol Connector_Generic:Conn_01x40
- added R?: 1K, symbol Device:R_Small
- added SW?: BOOTSEL, symbol Switch:SW_Push
- added SW?: RESET, symbol Switch:SW_Push
- added U?: RP2040, Package_DFN_QFN:QFN-56-1EP_7x7mm_P0.4mm_EP3.2x3.2mm, symbol MCU_RaspberryPi:RP2040
- added U?: W25Q32JVSS, Package_SO:SOIC-8_5.23x5.23mm_P1.27mm, symbol Memory_Flash:W25Q32JVSS
- added Y?: Crystal, symbol Device:Crystal
Connections:
- net GND: now also U?.61 (DCDC09_GND), C?.2, C?.2, C?.2, C?.2, C?.2, C?.2, C?.2, C?.2, J?.2 (Pin_2), J?.29 (Pin_29), J?.36 (Pin_36), SW?.1, SW?.2, U?.19 (TESTEN), U?.4 (GND)
- net PMEC_VDD: no longer U?.32 (VIN_3V3)
- net SYS_5V: now also J?.2 (Pin_2), J?.4 (Pin_4)
- net at U?.9 (I2Ct_SCL): no longer U?.16 (PA11/PA9)
- net at U?.10 (DBG_ACC): no longer U?.9 (PA2)
- net at U?.13 (PLUG_FLIP): no longer U?.10 (PA3)
- net at U?.17 (FAULT_IN): no longer U?.11 (PA4)
- net at U?.18 (SINK_EN): no longer U?.13 (PA6)
- net at U?.31 (PLUG_EVENT): no longer U?.14 (PA7)
- net at U?.6 (CAP_MIS): no longer U?.12 (PA5)
- net at U?.8 (I2Ct_SDA): no longer U?.17 (PA12/PA10)
- net LCD_B4: now reaches U?.15 (GPIO_P2_00)
- net LCD_B4: now also J?.25 (Pin_25)
- net LCD_B5: now reaches U?.16 (GPIO_P2_01)
- net LCD_B5: now also J?.26 (Pin_26)
- net LCD_B6: now reaches U?.17 (GPIO_P2_02)
- net LCD_B6: now also J?.27 (Pin_27)
- net LCD_B7: now reaches U?.18 (GPIO_P2_03)
- net LCD_B7: now also J?.28 (Pin_28)
- net LCD_G0: now reaches U?.19 (GPIO_P2_04)
- net LCD_G0: now also J?.13 (Pin_13)
- net LCD_G1: now reaches U?.20 (GPIO_P2_05)
- net LCD_G1: now also J?.14 (Pin_14)
- net LCD_G2: now reaches U?.21 (GPIO_P2_06)
- net LCD_G2: now also J?.15 (Pin_15)
- net LCD_G3: now reaches U?.22 (GPIO_P2_07)
- net LCD_G3: now also J?.16 (Pin_16)
- net IO_3V3: now reaches J?.1 (Pin_1)
- net at U?.33 (VDD09_A): now also U?.36 (VDD09_A), U?.57 (VDD09_A), C?.1, C?.1, C?.1, C?.1
- net LCD_B0: now reaches U?.11 (GPIO_P1_04)
- net LCD_B0: now also J?.21 (Pin_21)
- net LCD_B1: now reaches U?.12 (GPIO_P1_05)
- net LCD_B1: now also J?.22 (Pin_22)
- net LCD_B2: now reaches U?.13 (GPIO_P1_06)
- net LCD_B2: now also J?.23 (Pin_23)
- net LCD_B3: now reaches U?.14 (GPIO_P1_07)
- net LCD_B3: now also J?.24 (Pin_24)
- net LCD_R4: now reaches U?.37 (GPIO_P4_00)
- net LCD_R4: now also J?.9 (Pin_9)
- net LCD_R5: now reaches U?.38 (GPIO_P4_01)
- net LCD_R5: now also J?.10 (Pin_10)
- net LCD_R6: now reaches U?.39 (GPIO_P4_02)
- net LCD_R6: now also J?.11 (Pin_11)
- net LCD_R7: now reaches U?.40 (GPIO_P4_03)
- net LCD_R7: now also J?.12 (Pin_12)
- net LCD_HSYNC: now reaches U?.41 (GPIO_P4_04)
- net LCD_HSYNC: now also J?.32 (Pin_32)
- net LCD_VSYNC: now reaches U?.42 (GPIO_P4_05)
- net LCD_VSYNC: now also J?.33 (Pin_33)
- net LCD_DCLK: now reaches U?.43 (GPIO_P4_06)
- net LCD_DCLK: now also J?.30 (Pin_30)
- net LCD_DE: now reaches U?.44 (GPIO_P4_07)
- net LCD_DE: now also J?.31 (Pin_31), J?.34 (Pin_34)
- net LCD_G4: now reaches U?.25 (GPIO_P3_00)
- net LCD_G4: now also J?.17 (Pin_17)
- net LCD_G5: now reaches U?.26 (GPIO_P3_01)
- net LCD_G5: now also J?.18 (Pin_18)
- net LCD_G6: now reaches U?.27 (GPIO_P3_02)
- net LCD_G6: now also J?.19 (Pin_19)
- net LCD_G7: now reaches U?.28 (GPIO_P3_03)
- net LCD_G7: now also J?.20 (Pin_20)
- net LCD_R0: now reaches U?.29 (GPIO_P3_04)
- net LCD_R0: now also J?.5 (Pin_5)
- net LCD_R1: now reaches U?.30 (GPIO_P3_05)
- net LCD_R1: now also J?.6 (Pin_6)
- net LCD_R2: now reaches U?.31 (GPIO_P3_06)
- net LCD_R2: now also J?.7 (Pin_7)
- net LCD_R3: now reaches U?.32 (GPIO_P3_07)
- net LCD_R3: now also J?.8 (Pin_8)
- net PMEC_I2C_SCL: no longer names the net of U?.1 (PB7/PB8)
- new net: C?.1, U?.20 (XIN), Y?.1
- new net: C?.1, R?.1, Y?.2
- new net: R?.2, U?.21 (XOUT)
- new net: J?.1 (Pin_1), U?.24 (SWCLK)
- new net: J?.3 (Pin_3), U?.25 (SWD)
- new net: C?.1, C?.1, D?.1 (K), U?.8 (VCC)
- new net: J?.1 (Pin_1), U?.47 (USB_DP)
- new net: J?.2 (Pin_2), U?.46 (USB_DM)
- new net: U?.1 (IOVDD), U?.10 (IOVDD), U?.22 (IOVDD), U?.33 (IOVDD), U?.42 (IOVDD), U?.49 (IOVDD)
- new net: U?.23 (DVDD), U?.50 (DVDD)
- new net: SW?.2, U?.26 (RUN)
- new net EC_3V3: D?.2 (A)
- new net EC_QSPI_CLK: U?.52 (QSPI_SCLK), U?.6 (CLK)
- new net EC_QSPI_CS: SW?.1, U?.1 (~{CS}), U?.56 (QSPI_SS)
- new net EC_QSPI_IO0: U?.5 (DI(IO0)), U?.53 (QSPI_SD0)
- new net EC_QSPI_IO1: U?.2 (DO(IO1)), U?.55 (QSPI_SD1)
- new net EC_QSPI_IO2: U?.3 (IO2), U?.54 (QSPI_SD2)
- new net EC_QSPI_IO3: U?.51 (QSPI_SD3), U?.7 (IO3)
- no-connect marks 7 -> 8
Other:
- note added: "September 23, 2024 - October 7, 2024"
- note removed: "September 23, 2024"
- moved on the sheet: C?, L?, R?, U?, U?A, U?B, U?C, U?D, U?E, U?I, U?J
